File: BOB-PMW3610-SEIBOKU.kicad_pcb (KiCad board)
At the start: 2 copper layers, 30 x 20 mm, 17 parts, among them J1 Conn_02x04_Odd_Even, U1 TLV70019DDCR, U2 PMW3610DM-SUDU

Commit message: README.mdのタイトルを修正し、CHANGELOG.mdを追加
Other:
- board text added: "LENDS"
- board text added: "PMW3610 Breakout Board SEIBOKU rev1.2"
- board text removed: "pmw3610 breakout rev1.1"
